File: citizen_science_flora.brd (EAGLE design)
At the start: 86.6 x 79.6 mm, 118 parts, among them IC1 W25Q64JVXGIQ, J1 SM03B-SRSS-TB(LF)(SN), J2 TYPE-C-31-M-12, J4 60312202114511, J5 60312202114511, J6 TSM-102-02-S-SH, Q1 220mA/50V/3.5Ω, Q2 BSS138, U1 RP2350A, U10 PCF8563T/F4,118, U11 OPS-S56AAF5, U12 OPS-S56AAF5, U13 OPS-S56AAF5, U14 OPS-S56AAF5, U15 SN74LVC1T45DBVRG4, U2 APS6404L-3SQR-ZR, U3 ESP32-C3-MINI-1-N4, U4 MIC5504-3.3YM5-T5, U5 BME690, U6 ADM3260ARSZ, U7 ENS210-LQFM, U8 SFH6325-X017TEL0631, U9 AS3935-BQFT, Y1 12MHz

Commit message: Update citizen_science_flora.brd
Routing:
- net GND: track 0.00 -> 13.1 mm
- net 3.3V: track 73.6 -> 81.5 mm, vias 13 -> 15
- net N$16: track 0.00 -> 7.81 mm
- net N$15: track 0.00 -> 1.90 mm
Changed lines of the file:
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@@
 <attribute name="MF" value="ScioSense" x="7.8994" y="-44.069" size="1.778" layer="27" display="off"/>
 <attribute name="MP" value="ENS210-LQFM" x="7.8994" y="-44.069" size="1.778" layer="27" display="off"/>
-<attribute name="NAME" x="-29.9988" y="6.695" size="1.016" layer="25" font="vector" ratio="20"/>
+<attribute name="NAME" x="-24.7156" y="8.2444" size="1.016" layer="25" font="vector" ratio="20"/>
 <attribute name="PACKAGE" value="NON STANDARD-5 ScioSense" x="7.8994" y="-44.069" size="1.778" layer="27" display="off"/>
 <attribute name="PRICE" value="None" x="7.8994" y="-44.069" size="1.778" layer="27" display="off"/>
@@
 <vertex x="-41.9354" y="-19.2532"/>
 </polygon>
-<wire x1="-36.5506" y1="-0.2244" x2="-39.37" y2="-5.92" width="0" layer="19" extent="1-1"/>
-<wire x1="-35.306" y1="-0.0682" x2="-36.5506" y2="-0.2244" width="0" layer="19" extent="1-1"/>
-<wire x1="-33.812" y1="0.295" x2="-35.306" y2="-0.0682" width="0" layer="19" extent="1-1"/>
-<wire x1="-31.877" y1="1.27" x2="-31.552" y2="-0.665" width="0" layer="19" extent="1-1"/>
+<wire x1="-35.7124" y1="3.2432" x2="-34.0186" y2="3.2432" width="0.254" layer="1"/>
+<wire x1="-34.0186" y1="3.2432" x2="-33.9852" y2="3.2766" width="0.254" layer="1"/>
+<wire x1="-39.37" y1="-5.92" x2="-39.37" y2="-0.508" width="0.254" layer="1"/>
+<wire x1="-39.37" y1="-0.508" x2="-39.0652" y2="-0.2032" width="0.254" layer="1"/>
+<wire x1="-36.5718" y1="-0.2032" x2="-36.5506" y2="-0.2244" width="0.254" layer="1"/>
+<wire x1="-39.0652" y1="-0.2032" x2="-36.5718" y2="-0.2032" width="0.254" layer="1"/>
+<wire x1="-36.5506" y1="-0.2244" x2="-35.4622" y2="-0.2244" width="0.254" layer="1"/>
+<wire x1="-35.4622" y1="-0.2244" x2="-35.306" y2="-0.0682" width="0.254" layer="1"/>
+<wire x1="-35.306" y1="-0.0682" x2="-34.8408" y2="-0.0682" width="0.254" layer="1"/>
+<wire x1="-34.8408" y1="-0.0682" x2="-34.4678" y2="0.3048" width="0.254" layer="1"/>
+<wire x1="-34.4678" y1="0.3048" x2="-33.8218" y2="0.3048" width="0.254" layer="1"/>
+<wire x1="-33.8218" y1="0.3048" x2="-33.812" y2="0.295" width="0.254" layer="1"/>
+<wire x1="-31.552" y1="-0.665" x2="-31.877" y2="1.27" width="0" layer="19" extent="1-1"/>
+<wire x1="-33.812" y1="1.595" x2="-33.812" y2="0.295" width="0" layer="19" extent="1-1"/>
 <wire x1="15.1" y1="22.4865" x2="16.2734" y2="24.1046" width="0" layer="19" extent="1-1"/>
 <wire x1="3.384" y1="22.8284" x2="5.334" y2="24.0284" width="0" layer="19" extent="1-1"/>
-<wire x1="-35.7124" y1="3.2432" x2="-33.812" y2="1.595" width="0" layer="19" extent="1-1"/>
 <wire x1="12.7" y1="19.05" x2="15.1" y2="22.4865" width="0" layer="19" extent="1-1"/>
 </signal>
@@
 <wire x1="26.3144" y1="23.0632" x2="26.3398" y2="23.0378" width="0.2032" layer="15"/>
 <wire x1="26.3398" y1="23.0378" x2="26.3398" y2="22.3774" width="0.2032" layer="15"/>
+<wire x1="-27.3406" y1="8.476" x2="-29.505" y2="8.476" width="0.254" layer="1"/>
+<wire x1="-29.505" y1="8.476" x2="-29.5228" y2="8.4582" width="0.254" layer="1"/>
+<wire x1="-29.5228" y1="8.4582" x2="-29.5228" y2="7.9168" width="0.254" layer="1"/>
+<wire x1="-29.5228" y1="7.9168" x2="-29.845" y2="7.5946" width="0.254" layer="1"/>
+<via x="-29.845" y="7.5946" extent="1-16" drill="0.381"/>
+<wire x1="-29.845" y1="7.5946" x2="-30.4546" y2="7.5946" width="0.254" layer="15"/>
+<wire x1="-30.4546" y1="7.5946" x2="-30.48" y2="7.62" width="0.254" layer="15"/>
+<wire x1="-32.852" y1="3.205" x2="-32.852" y2="4.4606" width="0.254" layer="1"/>
+<wire x1="-32.852" y1="4.4606" x2="-32.766" y2="4.5466" width="0.254" layer="1"/>
+<wire x1="-32.766" y1="4.5466" x2="-32.2072" y2="4.5466" width="0.254" layer="1"/>
+<wire x1="-32.202" y1="4.5414" x2="-32.202" y2="3.205" width="0.254" layer="1"/>
+<wire x1="-32.2072" y1="4.5466" x2="-32.202" y2="4.5414" width="0.254" layer="1"/>
+<via x="-32.202" y="4.5414" extent="1-16" drill="0.381"/>
+<wire x1="-32.202" y1="4.5414" x2="-32.202" y2="5.1764" width="0.254" layer="15"/>
+<wire x1="-32.202" y1="5.1764" x2="-32.258" y2="5.2324" width="0.254" layer="15"/>
 <wire x1="37.3888" y1="8.5132" x2="38.608" y2="8.517" width="0" layer="19" extent="1-1"/>
 <wire x1="38.562" y1="6.789" x2="38.608" y2="8.517" width="0" layer="19" extent="1-1"/>
@@
 <wire x1="-26.8406" y1="30.335575" x2="-27.17" y2="22.86" width="0" layer="19" extent="1-1"/>
 <wire x1="-27.3406" y1="8.476" x2="-18.2118" y2="18.8538" width="0" layer="19" extent="1-1"/>
-<wire x1="-29.5228" y1="8.4582" x2="-27.3406" y2="8.476" width="0" layer="19" extent="1-1"/>
-<wire x1="-26.2048" y1="3.6322" x2="-27.3406" y2="8.476" width="0" layer="19" extent="1-1"/>
-<wire x1="-27.6414" y1="2.4446" x2="-26.2048" y2="3.6322" width="0" layer="19" extent="1-1"/>
-<wire x1="-27.6414" y1="0.8446" x2="-27.6414" y2="2.4446" width="0" layer="19" extent="1-1"/>
-<wire x1="-28.702" y1="0.8462" x2="-27.6414" y2="0.8446" width="0" layer="19" extent="1-1"/>
-<wire x1="-29.942" y1="0.295" x2="-28.702" y2="0.8462" width="0" layer="19" extent="1-1"/>
+<wire x1="-32.258" y1="5.2324" x2="-30.48" y2="7.62" width="0" layer="19" extent="15-15"/>
+<wire x1="-29.942" y1="0.295" x2="-32.202" y2="3.205" width="0" layer="19" extent="1-1"/>
+<wire x1="-28.702" y1="0.8462" x2="-29.942" y2="0.295" width="0" layer="19" extent="1-1"/>
+<wire x1="-27.6414" y1="0.8446" x2="-28.702" y2="0.8462" width="0" layer="19" extent="1-1"/>
+<wire x1="-27.6414" y1="2.4446" x2="-27.6414" y2="0.8446" width="0" layer="19" extent="1-1"/>
+<wire x1="-26.2048" y1="3.6322" x2="-27.6414" y2="2.4446" width="0" layer="19" extent="1-1"/>
 <wire x1="-25.2414" y1="1.6446" x2="-26.2048" y2="3.6322" width="0" layer="19" extent="1-1"/>
 <wire x1="-32.202" y1="-0.665" x2="-29.942" y2="0.295" width="0" layer="19" extent="1-1"/>
 <wire x1="-32.852" y1="-0.665" x2="-32.202" y2="-0.665" width="0" layer="19" extent="1-1"/>
 <wire x1="-32.4358" y1="-2.7474" x2="-32.202" y2="-0.665" width="0" layer="19" extent="1-1"/>
-<wire x1="-32.202" y1="3.205" x2="-29.942" y2="0.295" width="0" layer="19" extent="1-1"/>
-<wire x1="-32.852" y1="3.205" x2="-32.202" y2="3.205" width="0" layer="19" extent="1-1"/>
 <wire x1="-28.3972" y1="-6.9892" x2="-32.4358" y2="-2.7474" width="0" layer="19" extent="1-1"/>
 <wire x1="-27.0002" y1="-6.9892" x2="-28.3972" y2="-6.9892" width="0" layer="19" extent="1-1"/>
@@
 <contactref element="U9" pad="1"/>
 <contactref element="C31" pad="1"/>
-<wire x1="-33.812" y1="2.245" x2="-35.7124" y2="2.2432" width="0" layer="19" extent="1-1"/>
+<wire x1="-35.7124" y1="2.2432" x2="-33.8138" y2="2.2432" width="0.254" layer="1"/>
+<wire x1="-33.8138" y1="2.2432" x2="-33.812" y2="2.245" width="0.254" layer="1"/>
 </signal>
 <signal name="N$16">
@@
 <contactref element="C33" pad="1"/>
 <contactref element="R18" pad="2"/>
-<wire x1="-36.5506" y1="0.9356" x2="-39.37" y2="3.38" width="0" layer="19" extent="1-1"/>
-<wire x1="-35.306" y1="0.9318" x2="-36.5506" y2="0.9356" width="0" layer="19" extent="1-1"/>
-<wire x1="-33.812" y1="0.945" x2="-35.306" y2="0.9318" width="0" layer="19" extent="1-1"/>
+<wire x1="-33.812" y1="0.945" x2="-35.2928" y2="0.945" width="0.254" layer="1"/>
+<wire x1="-35.2928" y1="0.945" x2="-35.306" y2="0.9318" width="0.254" layer="1"/>
+<wire x1="-35.306" y1="0.9318" x2="-35.3098" y2="0.9356" width="0.254" layer="1"/>
+<wire x1="-35.3098" y1="0.9356" x2="-36.5506" y2="0.9356" width="0.254" layer="1"/>
+<wire x1="-36.5506" y1="0.9356" x2="-39.0356" y2="0.9356" width="0.254" layer="1"/>
+<wire x1="-39.0356" y1="0.9356" x2="-39.37" y2="1.27" width="0.254" layer="1"/>
+<wire x1="-39.37" y1="1.27" x2="-39.37" y2="3.38" width="0.254" layer="1"/>
 </signal>
 <signal name="VCC-ISO">

Commit message: Update citizen_science_flora.brd
Parts:
- moved C26 11.6 mm to (-32.0, -6.05), turned to 180 degrees
- moved U5 7.38 mm to (-29.0, -5.66)
- moved C27 6.66 mm to (-32.0, -4.42), turned to 180 degrees
- moved R11 5.55 mm to (-24.3, -11.3), turned to 0 degrees
- moved R12 1.88 mm to (-25.2, -8.18), turned to 0 degrees
- moved C32 1.40 mm to (-33.5, -2.36), turned to 180 degrees
- moved C25 0.86 mm to (-33.0, -12.2), turned to 270 degrees
Routing:
- net 3.3V: track 81.5 -> 103.5 mm, vias 15 -> 18
- net SCL: track 0.00 -> 4.92 mm
- net SDA: track 0.00 -> 4.77 mm
- net GND: track 13.1 -> 15.1 mm

Commit message: Update citizen_science_flora.brd
Parts:
- moved C28 7.83 mm to (-19.5, 26.1), turned to 240 degrees
Routing:
- net 3.3V: track 103.5 -> 126.0 mm, vias 18 -> 21
- net V_USB: track 9.24 -> 12.0 mm
Changed lines of the file:
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@@
 </layers>
 <board>
-<fusionsync huburn="a.cGVyc29uYWw6dWUyOTBlYmM4" projecturn="a.cGVyc29uYWw6dWUyOTBlYmM4IzIwMjQwNTE5NzY3MjkwODMx" f3durn="urn:adsk.wipprod:dm.lineage:hKbjeZyhTQCGIgAsdv3kWg" pcbguid="" lastpulledtime="" lastsyncedchangeguid="" latestrevisionid="eaa05dbf-31ce-40a9-a6cf-c28e765d50ed" lastsyncedrevisionid="eaa05dbf-31ce-40a9-a6cf-c28e765d50ed" lastboardhashguid="2cc016ec-c287-fb01-aef3-a2e37659a8d4" lastpushedtime="2025-01-05T07:56:31Z" linktopcb3d="true"/>
+<fusionsync huburn="a.cGVyc29uYWw6dWUyOTBlYmM4" projecturn="a.cGVyc29uYWw6dWUyOTBlYmM4IzIwMjQwNTE5NzY3MjkwODMx" f3durn="urn:adsk.wipprod:dm.lineage:hKbjeZyhTQCGIgAsdv3kWg" pcbguid="" lastpulledtime="" lastsyncedchangeguid="" latestrevisionid="5b8a528c-b45a-4ea4-8c99-216c39175609" lastsyncedrevisionid="5b8a528c-b45a-4ea4-8c99-216c39175609" lastboardhashguid="1f314a6d-59e9-339e-f35d-d5c104a4aea2" lastpushedtime="2025-01-06T07:51:02Z" linktopcb3d="true"/>
 <plain>
 <polygon width="0.1524" layer="30">
@@
 <attribute name="VALUE" x="-32.0294" y="-3.8576" size="0.6096" layer="27" font="vector" ratio="20" rot="R180" align="top-center"/>
 </element>
-<element name="C28" library="SparkFun-Capacitors" library_urn="urn:adsk.eagle:library:510" package="0402-TIGHT" package3d_urn="urn:adsk.eagle:package:41385069/1" override_package3d_urn="urn:adsk.eagle:package:46141828/2" override_package_urn="urn:adsk.eagle:footprint:41385056/1" value="0.1uF" x="-26.67" y="22.86" smashed="yes">
-<attribute name="NAME" x="-27.051" y="21.136" size="1.016" layer="25" font="vector" ratio="20" align="bottom-center"/>
-<attribute name="PROD_ID" value="CAP-16507" x="7.62" y="-57.15" size="1.778" layer="27" display="off"/>
-<attribute name="VALUE" x="-26.67" y="22.298" size="0.6096" layer="27" font="vector" ratio="20" align="top-center"/>
+<element name="C28" library="SparkFun-Capacitors" library_urn="urn:adsk.eagle:library:510" package="0402-TIGHT" package3d_urn="urn:adsk.eagle:package:41385069/1" override_package3d_urn="urn:adsk.eagle:package:46141828/2" override_package_urn="urn:adsk.eagle:footprint:41385056/1" value="0.1uF" x="-19.5326" y="26.0858" smashed="yes" rot="R240">
+<attribute name="NAME" x="-20.708125" y="24.255153125" size="1.016" layer="25" font="vector" ratio="20" rot="R240" align="bottom-center"/>
+<attribute name="PROD_ID" value="CAP-16507" x="-105.968290625" y="36.3947875" size="1.778" layer="27" rot="R240" display="off"/>
+<attribute name="VALUE" x="-20.01930625" y="26.3668" size="0.6096" layer="27" font="vector" ratio="20" rot="R240" align="top-center"/>
 </element>
 <element name="C29" library="SparkFun-Capacitors" library_urn="urn:adsk.eagle:library:510" package="0402-TIGHT" package3d_urn="urn:adsk.eagle:package:41385069/1" override_package3d_urn="urn:adsk.eagle:package:46141977/2" override_package_urn="urn:adsk.eagle:footprint:41385056/1" value="0.1uF" x="-30.0228" y="8.4582" smashed="yes" rot="R180">
@@
 <via x="-33.147" y="-10.6934" extent="1-16" drill="0.381"/>
 <wire x1="-33.147" y1="-10.6934" x2="-33.147" y2="-9.9568" width="0.254" layer="15"/>
+<wire x1="-18.2118" y1="18.8538" x2="-14.1662" y2="18.8538" width="0.254" layer="1"/>
+<wire x1="-14.1662" y1="18.8538" x2="-13.97" y2="19.05" width="0.254" layer="1"/>
+<wire x1="-13.97" y1="19.05" x2="-14.4168" y2="19.05" width="0.254" layer="1"/>
+<wire x1="-14.4168" y1="19.05" x2="-14.6252" y2="18.8416" width="0.254" layer="1"/>
+<wire x1="-14.6252" y1="18.8416" x2="-12.4408" y2="18.8416" width="0.254" layer="1"/>
+<wire x1="-12.4408" y1="18.8416" x2="-12.0904" y2="18.4912" width="0.254" layer="1"/>
+<via x="-12.0904" y="18.4912" extent="1-16" drill="0.381"/>
+<wire x1="-12.0904" y1="18.4912" x2="-11.7348" y2="18.1356" width="0.254" layer="15"/>
+<wire x1="-11.7348" y1="18.1356" x2="-10.9728" y2="18.1356" width="0.254" layer="15"/>
+<wire x1="-19.2826" y1="26.5188125" x2="-21.69299375" y2="27.736053125" width="0.254" layer="1"/>
+<wire x1="-21.69299375" y1="27.736053125" x2="-26.8406" y2="30.335575" width="0.254" layer="1"/>
+<wire x1="-19.2826" y1="26.5188125" x2="-18.9992" y2="27.2542" width="0.254" layer="1"/>
+<via x="-18.9992" y="27.2542" extent="1-16" drill="0.381"/>
+<wire x1="-18.9992" y1="27.2542" x2="-19.2786" y2="26.5684" width="0.254" layer="15"/>
+<wire x1="0.975" y1="-15.45" x2="0.9652" y2="-13.5302" width="0.254" layer="1"/>
+<wire x1="0.9652" y1="-13.5302" x2="0.2286" y2="-13.5636" width="0.254" layer="1"/>
+<via x="0.2286" y="-13.5636" extent="1-16" drill="0.381"/>
+<wire x1="0.2286" y1="-13.5636" x2="-0.6858" y2="-13.5382" width="0.254" layer="15"/>
 <wire x1="37.3888" y1="8.5132" x2="38.608" y2="8.517" width="0" layer="19" extent="1-1"/>
 <wire x1="38.562" y1="6.789" x2="38.608" y2="8.517" width="0" layer="19" extent="1-1"/>
@@
 <wire x1="12.5222" y1="-13.5574" x2="19.1474" y2="-14.8844" width="0" layer="19" extent="1-1"/>
 <wire x1="0.975" y1="-15.45" x2="11.0156" y2="-14.8844" width="0" layer="19" extent="1-1"/>
-<wire x1="0.9652" y1="-13.5302" x2="0.975" y2="-15.45" width="0" layer="19" extent="1-1"/>
 <wire x1="21.5688" y1="11.9634" x2="27.94" y2="-2.54" width="0" layer="19" extent="1-15"/>
 <wire x1="19.9492" y1="13.1422" x2="21.5688" y2="11.9634" width="0" layer="19" extent="1-1"/>
@@
 <wire x1="0.4614" y1="26.8224" x2="2.3114" y2="29.7646" width="0" layer="19" extent="1-1"/>
 <wire x1="-7.3406" y1="23.6912" x2="0.4614" y2="26.8224" width="0" layer="19" extent="1-1"/>
-<wire x1="-14.6252" y1="18.8416" x2="-7.3406" y2="23.6912" width="0" layer="19" extent="1-1"/>
-<wire x1="-18.2118" y1="18.8538" x2="-14.6252" y2="18.8416" width="0" layer="19" extent="1-1"/>
-<wire x1="-27.17" y1="22.86" x2="-18.2118" y2="18.8538" width="0" layer="19" extent="1-1"/>
-<wire x1="-26.8406" y1="30.335575" x2="-27.17" y2="22.86" width="0" layer="19" extent="1-1"/>
+<wire x1="-10.9728" y1="18.1356" x2="-7.3406" y2="23.6912" width="0" layer="19" extent="1-15"/>
+<wire x1="-19.2826" y1="26.5188125" x2="-18.2118" y2="18.8538" width="0" layer="19" extent="1-1"/>
 <wire x1="-27.3406" y1="8.476" x2="-18.2118" y2="18.8538" width="0" layer="19" extent="1-1"/>
 <wire x1="-32.258" y1="5.2324" x2="-30.48" y2="7.62" width="0" layer="19" extent="15-15"/>
@@
 <wire x1="20.513" y1="25.4864" x2="20.8788" y2="25.1206" width="0.2032" layer="1"/>
 <wire x1="20.8788" y1="25.1206" x2="22.1742" y2="25.1206" width="0.2032" layer="1"/>
+<wire x1="-2.275" y1="-15.45" x2="-2.3702" y2="-13.6398" width="0.254" layer="1"/>
+<wire x1="-2.3702" y1="-13.6398" x2="-2.3702" y2="-12.7" width="0.254" layer="1"/>
 <wire x1="23.7062" y1="26.3906" x2="24.3078" y2="27.7114" width="0" layer="19" extent="1-1"/>
 <wire x1="19.9492" y1="10.6322" x2="20.513" y2="26.311" width="0" layer="19" extent="1-1"/>
@@
 <wire x1="6.0452" y1="-10.6002" x2="6.3204" y2="-12.9794" width="0" layer="19" extent="1-1"/>
 <wire x1="-2.3702" y1="-12.7" x2="6.0452" y2="-10.6002" width="0" layer="19" extent="1-1"/>
-<wire x1="-2.3702" y1="-13.6398" x2="-2.3702" y2="-12.7" width="0" layer="19" extent="1-1"/>
-<wire x1="-2.275" y1="-15.45" x2="-2.3702" y2="-13.6398" width="0" layer="19" extent="1-1"/>
 <wire x1="-4.7286" y1="-17.145" x2="-2.275" y2="-15.45" width="0" layer="19" extent="1-1"/>
 <wire x1="-6.278" y1="-13.1064" x2="-2.3702" y2="-12.7" width="0" layer="19" extent="1-1"/>

Commit message: Update citizen_science_flora.brd
Routing:
- net 3.3V: track 126.0 -> 140.1 mm, vias 21 -> 23
- added copper zone on layer 15, net 3.3V
Changed lines of the file:
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@@
 <via x="0.2286" y="-13.5636" extent="1-16" drill="0.381"/>
 <wire x1="0.2286" y1="-13.5636" x2="-0.6858" y2="-13.5382" width="0.254" layer="15"/>
-<wire x1="37.3888" y1="8.5132" x2="38.608" y2="8.517" width="0" layer="19" extent="1-1"/>
-<wire x1="38.562" y1="6.789" x2="38.608" y2="8.517" width="0" layer="19" extent="1-1"/>
-<wire x1="29.1084" y1="-3.4756" x2="38.562" y2="6.789" width="0" layer="19" extent="1-1"/>
-<wire x1="19.1474" y1="-14.8844" x2="27.9146" y2="-3.2766" width="0" layer="19" extent="1-1"/>
-<wire x1="12.5222" y1="-13.5574" x2="19.1474" y2="-14.8844" width="0" layer="19" extent="1-1"/>
-<wire x1="0.975" y1="-15.45" x2="11.0156" y2="-14.8844" width="0" layer="19" extent="1-1"/>
-<wire x1="21.5688" y1="11.9634" x2="27.94" y2="-2.54" width="0" layer="19" extent="1-15"/>
-<wire x1="19.9492" y1="13.1422" x2="21.5688" y2="11.9634" width="0" layer="19" extent="1-1"/>
-<wire x1="18.9992" y1="10.6322" x2="19.9492" y2="13.1422" width="0" layer="19" extent="1-1"/>
-<wire x1="18.7278" y1="15.5448" x2="19.9492" y2="13.1422" width="0" layer="19" extent="1-1"/>
-<wire x1="17.78" y1="19.05" x2="17.78" y2="17.78" width="0" layer="19" extent="15-15"/>
-<wire x1="20.011" y1="20.7772" x2="18.7532" y2="19.6088" width="0" layer="19" extent="1-1"/>
-<wire x1="14.3" y1="22.4865" x2="16.1365" y2="21.85" width="0" layer="19" extent="1-1"/>
-<wire x1="12.7" y1="22.4865" x2="14.3" y2="22.4865" width="0" layer="19" extent="1-1"/>
+<wire x1="18.9992" y1="10.6322" x2="18.9992" y2="11.7602" width="0.254" layer="1"/>
+<wire x1="19.9492" y1="13.1422" x2="19.9492" y2="12.3088" width="0.254" layer="1"/>
+<wire x1="19.9492" y1="12.3088" x2="20.1168" y2="12.1412" width="0.254" layer="1"/>
+<wire x1="20.1168" y1="12.1412" x2="20.2946" y2="11.9634" width="0.254" layer="1"/>
+<wire x1="20.2946" y1="11.9634" x2="21.5688" y2="11.9634" width="0.254" layer="1"/>
+<wire x1="18.9992" y1="11.7602" x2="19.3802" y2="12.1412" width="0.254" layer="1"/>
+<wire x1="19.3802" y1="12.1412" x2="20.1168" y2="12.1412" width="0.254" layer="1"/>
+<wire x1="19.9492" y1="13.1422" x2="19.9492" y2="14.1834" width="0.254" layer="1"/>
+<wire x1="20.2692" y1="14.5034" x2="20.447" y2="14.5034" width="0.254" layer="1"/>
+<via x="20.447" y="14.5034" extent="1-16" drill="0.381"/>
+<wire x1="20.447" y1="14.5034" x2="21.3614" y2="14.5034" width="0.254" layer="15"/>
+<wire x1="21.3614" y1="14.5034" x2="21.6154" y2="14.2494" width="0.254" layer="15"/>
+<wire x1="19.9492" y1="14.1834" x2="20.2692" y2="14.5034" width="0.254" layer="1"/>
+<wire x1="38.562" y1="6.789" x2="38.562" y2="8.471" width="0.254" layer="1"/>
+<wire x1="38.562" y1="8.471" x2="38.608" y2="8.517" width="0.254" layer="1"/>
+<wire x1="38.608" y1="8.517" x2="37.3926" y2="8.517" width="0.254" layer="1"/>
+<wire x1="37.3926" y1="8.517" x2="37.3888" y2="8.5132" width="0.254" layer="1"/>
+<wire x1="37.3888" y1="8.5132" x2="36.521" y2="8.5132" width="0.254" layer="1"/>
+<wire x1="36.521" y1="8.5132" x2="36.2712" y2="8.763" width="0.254" layer="1"/>
+<via x="36.2712" y="8.763" extent="1-16" drill="0.381"/>
+<wire x1="36.2712" y1="8.763" x2="36.195" y2="8.8392" width="0.254" layer="15"/>
+<wire x1="36.195" y1="8.8392" x2="36.195" y2="9.8044" width="0.254" layer="15"/>
+<wire x1="22.1742" y1="20.7772" x2="22.4028" y2="20.7772" width="0.254" layer="15"/>
+<wire x1="22.4028" y1="20.7772" x2="22.86" y2="20.32" width="0.254" layer="15"/>
+<polygon width="0.254" layer="15">
+<vertex x="-41.91" y="-19.05"/>
+<vertex x="-41.91" y="-7.1882"/>
+<vertex x="-41.8592" y="-7.1374"/>
+<vertex x="-34.671" y="-7.1374"/>
+<vertex x="-34.671" y="-5.461"/>
+<vertex x="-34.671" y="4.699"/>
+<vertex x="-35.306" y="4.699"/>
+<vertex x="-46.5074" y="4.699"/>
+<vertex x="-46.5074" y="40.5384"/>
+<vertex x="46.99" y="40.5384"/>
+<vertex x="46.99" y="39.116"/>
+<vertex x="46.99" y="7.5692"/>
+<vertex x="41.8846" y="7.5692"/>
+<vertex x="41.8846" y="-16.9926"/>
+<vertex x="39.9288" y="-16.9926"/>
+<vertex x="7.5946" y="-16.9926"/>
+<vertex x="6.5024" y="-18.0848"/>
+<vertex x="6.0452" y="-18.0848"/>
+<vertex x="-6.35" y="-18.0848"/>
+<vertex x="-6.3754" y="-18.0594"/>
+<vertex x="-6.5532" y="-18.0594"/>
+<vertex x="-7.5438" y="-19.05"/>
+<vertex x="-41.8592" y="-19.05"/>
+</polygon>
+<wire x1="-24.6422" y1="-8.1788" x2="-23.7278" y2="-11.3284" width="0" layer="19" extent="1-1"/>
+<wire x1="-27.8322" y1="-5.2642" x2="-24.6422" y2="-8.1788" width="0" layer="19" extent="1-1"/>
 <wire x1="8.5424" y1="25.273" x2="10.9474" y2="25.3826" width="0" layer="19" extent="1-1"/>
-<wire x1="9.2635" y1="21.85" x2="12.3" y2="22.4865" width="0" layer="19" extent="1-1"/>
-<wire x1="7.0358" y1="18.5166" x2="6.5603625" y2="20.5849" width="0" layer="19" extent="1-1"/>
-<wire x1="5.5922" y1="16.6878" x2="6.9262" y2="17.8562" width="0" layer="19" extent="1-1"/>
-<wire x1="6.9596" y1="12.9286" x2="5.5118" y2="15.7226" width="0" layer="19" extent="1-15"/>
-<wire x1="7.9328" y1="28.6004" x2="8.5424" y2="25.273" width="0" layer="19" extent="1-1"/>
+<wire x1="-29.942" y1="0.295" x2="-32.202" y2="-0.665" width="0" layer="19" extent="1-1"/>
 <wire x1="2.3114" y1="29.7646" x2="6.711" y2="28.6138" width="0" layer="19" extent="1-1"/>
 <wire x1="0.4614" y1="26.8224" x2="2.3114" y2="29.7646" width="0" layer="19" extent="1-1"/>
-<wire x1="-7.3406" y1="23.6912" x2="0.4614" y2="26.8224" width="0" layer="19" extent="1-1"/>
-<wire x1="-10.9728" y1="18.1356" x2="-7.3406" y2="23.6912" width="0" layer="19" extent="1-15"/>
-<wire x1="-19.2826" y1="26.5188125" x2="-18.2118" y2="18.8538" width="0" layer="19" extent="1-1"/>
-<wire x1="-27.3406" y1="8.476" x2="-18.2118" y2="18.8538" width="0" layer="19" extent="1-1"/>
-<wire x1="-32.258" y1="5.2324" x2="-30.48" y2="7.62" width="0" layer="19" extent="15-15"/>
-<wire x1="-29.942" y1="0.295" x2="-32.202" y2="3.205" width="0" layer="19" extent="1-1"/>
-<wire x1="-32.202" y1="-0.665" x2="-29.942" y2="0.295" width="0" layer="19" extent="1-1"/>
-<wire x1="-30.2322" y1="-6.0642" x2="-30.2322" y2="-4.4642" width="0" layer="19" extent="1-1"/>
-<wire x1="-33.147" y1="-9.9568" x2="-32.4104" y2="-6.9088" width="0" layer="19" extent="15-15"/>
-<wire x1="-24.6422" y1="-8.1788" x2="-27.8322" y2="-5.2642" width="0" layer="19" extent="1-1"/>
-<wire x1="-23.7278" y1="-11.3284" x2="-24.6422" y2="-8.1788" width="0" layer="19" extent="1-1"/>
+<wire x1="-7.3406" y1="23.6912" x2="-10.9728" y2="18.1356" width="0" layer="19" extent="1-15"/>
+<wire x1="19.1474" y1="-14.8844" x2="12.5222" y2="-13.5574" width="0" layer="19" extent="1-1"/>
 </signal>
 <signal name="N$1">
