File: citizen_science_flora.brd (EAGLE design)
At the start: 86.6 x 79.6 mm, 118 parts, among them IC1 W25Q64JVXGIQ, J1 SM03B-SRSS-TB(LF)(SN), J2 TYPE-C-31-M-12, J4 60312202114511, J5 60312202114511, J6 TSM-102-02-S-SH, Q1 220mA/50V/3.5Ω, Q2 BSS138, U1 RP2350A, U10 PCF8563T/F4,118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

Commit message: Update citizen_science_flora.brd
Parts:
- moved R23 0.56 mm to (-5.28, -16.6), turned to 90 degrees
- moved C52 0.35 mm to (-18.7, -13.3)
- moved C51 0.35 mm to (-7.19, -13.2)
Routing:
- net V_USB: track 12.0 -> 127.9 mm, vias 0 -> 6
- net !FLASH_CS: track 1.90 -> 18.5 mm, vias 0 -> 2
- net !USB_BOOT: track 4.10 -> 19.2 mm, vias 0 -> 2
- net QSPI_CLK: track 6.92 -> 20.0 mm, vias 1 -> 2
- net 3.3V: track 140.1 -> 152.3 mm, vias 23 -> 27
- net PDIS: track 0.00 -> 7.59 mm
- net GND: track 15.1 -> 17.6 mm

Commit message: Update citizen_science_flora.brd
Routing:
- net SCL_ISO: track 0.00 -> 47.3 mm, vias 0 -> 2
- net SDA_ISO: track 0.00 -> 40.8 mm, vias 0 -> 2
- net !ESP32_BOOT: track 0.00 -> 37.7 mm, vias 0 -> 2
- net ESP32_MOSI: track 0.00 -> 35.8 mm, vias 0 -> 2
- net ESP32_CS: track 0.00 -> 35.5 mm, vias 0 -> 2
- net ESP32_SCK: track 0.00 -> 33.5 mm, vias 0 -> 2
- net ESP32_MISO: track 0.00 -> 31.1 mm, vias 0 -> 2
- net ESP32_HANDSHAKE: track 0.00 -> 31.0 mm, vias 0 -> 2
- net INT_SOIL_ISO: track 0.00 -> 30.4 mm, vias 0 -> 2
- net !RESET: track 0.00 -> 29.2 mm, vias 0 -> 2
- net VCC-ISO: track 0.00 -> 27.2 mm, vias 0 -> 7
- net SWCLK: track 0.00 -> 26.5 mm, vias 0 -> 2
- net SWDIO: track 0.00 -> 25.2 mm, vias 0 -> 2
- net INT_SOILTEMP_ISO: track 0.00 -> 24.2 mm
- net PRB1: track 0.00 -> 13.7 mm
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
Commit message: Update citizen_science_flora.brd
Routing:
- net SD_CLK: track 0.00 -> 59.0 mm, vias 0 -> 2
- net SWITCH: track 0.00 -> 55.1 mm, vias 0 -> 2
- net CMD: track 0.00 -> 54.8 mm, vias 0 -> 2
- net DAT3: track 0.00 -> 53.1 mm, vias 0 -> 2
- net DAT0: track 0.00 -> 51.8 mm, vias 0 -> 2
- net DAT2: track 0.00 -> 51.4 mm
- net DAT1: track 0.00 -> 51.3 mm, vias 0 -> 2
- net SCL: track 4.92 -> 54.1 mm, vias 0 -> 2
- net SDA: track 4.77 -> 53.3 mm, vias 0 -> 2
- net INT_RTC: track 0.00 -> 41.7 mm, vias 0 -> 2
- net !ESP32_RST: track 0.00 -> 33.8 mm, vias 0 -> 2
- net 1.1V: track 30.4 -> 41.5 mm
- net NEOPIXEL_3.3V: track 0.00 -> 5.57 mm
- net N$26: track 3.24 -> 8.07 mm
- net !RESET: track 29.2 -> 34.0 mm
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
Commit message: Update citizen_science_flora.brd
Parts:
- moved C15 4.56 mm to (2.24, 18.0), turned to 270 degrees
Routing:
- net SDA: track 53.3 -> 216.1 mm, vias 2 -> 5
- net ESP32_TX: track 0.00 -> 112.2 mm, vias 0 -> 2
- net ESP32_RX: track 0.00 -> 111.5 mm, vias 0 -> 2
- net SCL: track 54.1 -> 154.5 mm, vias 2 -> 4
- net INT_SOILTEMP: track 4.73 -> 66.6 mm, vias 0 -> 2
- net PDIS_EN: track 2.99 -> 61.6 mm, vias 0 -> 3
- net IRQ_LIGHTNING: track 0.00 -> 56.9 mm, vias 0 -> 2
- net INT_SOIL: track 6.77 -> 62.5 mm, vias 0 -> 2
- net BUZZER_DRIVER: track 0.00 -> 37.4 mm, vias 0 -> 2
- net N$22: track 0.00 -> 35.6 mm
- net N$24: track 0.00 -> 35.3 mm
- net N$23: track 0.00 -> 35.0 mm
- net N$25: track 4.10 -> 20.0 mm
- net 1.1V: track 41.5 -> 48.1 mm
- net GND: track 19.2 -> 22.1 mm, vias 3 -> 9
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