File: citizen_science_flora.brd (EAGLE design)
At the start: 86.6 x 79.6 mm, 118 parts, among them IC1 W25Q64JVXGIQ, J1 SM03B-SRSS-TB(LF)(SN), J2 TYPE-C-31-M-12, J4 60312202114511, J5 60312202114511, J6 TSM-102-02-S-SH, Q1 220mA/50V/3.5Ω, Q2 BSS138, U1 RP2350A, U10 PCF8563T/F4,118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

Commit message: updated gerber files
Parts:
- removed L1: 3.3µH, SparkFun-Coils:0805
- added L4: 3.3uH, LQH2MCN120K02L:IND_LQH2MCN120K02L
- moved C11 0.43 mm to (15.4, 25.1)
- moved C12 0.17 mm to (15.9, 24.2)
Connections:
- net 1.1V: now also L4.2; no longer L1.2
- net N$2: now also L4.1; no longer L1.1
Routing:
- net GND: track 22.1 -> 23.7 mm
- net N$2: track 8.36 -> 6.75 mm
- net 3.3V: track 151.8 -> 150.8 mm
