File: citizen_science_flora.sch (EAGLE design)
At the start: 118 parts, among them IC1 W25Q64JVXGIQ, J1 SM03B-SRSS-TB(LF)(SN), J2 TYPE-C-31-M-12, J4 60312202114511, J5 60312202114511, J6 TSM-102-02-S-SH, Q1 220mA/50V/3.5Ω, Q2 BSS138, U1 RP2350A, U10 PCF8563T/F4,118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

Commit message: updated gerber files
Parts:
- removed L1: 3.3µH, SparkFun-Coils:INDUCTOR-0805-3.3UH
- added L4: 3.3uH, LQH2MCN120K02L:LQH2MCN120K02L
Connections:
- net 1.1V: now also L4.P$2; no longer L1.2
- net N$2: now also L4.P$1; no longer L1.1
Changed lines of the file:
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@@
 <part name="GND4" library="SparkFun-PowerSymbols" library_urn="urn:adsk.eagle:library:530" deviceset="GND" device=""/>
 <part name="R1" library="SparkFun-Resistors" library_urn="urn:adsk.eagle:library:532" deviceset="33OHM" device="-0402-1/10W-1%" package3d_urn="urn:adsk.eagle:package:39657/2" override_package3d_urn="urn:adsk.eagle:package:46143275/2" override_package_urn="urn:adsk.eagle:footprint:39625/2" value="33"/>
-<part name="L1" library="SparkFun-Coils" library_urn="urn:adsk.eagle:library:512" deviceset="INDUCTOR" device="-0805-3.3UH" package3d_urn="urn:adsk.eagle:package:37579/2" override_package3d_urn="urn:adsk.eagle:package:46143259/2" override_package_urn="urn:adsk.eagle:footprint:37561/2" value="3.3µH"/>
 <part name="SUPPLY3" library="SparkFun-PowerSymbols" library_urn="urn:adsk.eagle:library:530" deviceset="1.1V" device=""/>
 <part name="C11" library="SparkFun-Capacitors" library_urn="urn:adsk.eagle:library:510" deviceset="4.7UF" device="-0402_TIGHT-6.3V-20%-X5R" package3d_urn="urn:adsk.eagle:package:41385069/1" override_package3d_urn="urn:adsk.eagle:package:46141773/2" override_package_urn="urn:adsk.eagle:footprint:41385056/1" value="4.7uF"/>
@@
 <part name="C52" library="SparkFun-Capacitors" library_urn="urn:adsk.eagle:library:510" deviceset="0.1UF" device="-0402-6.3V-10%-X7R" package3d_urn="urn:adsk.eagle:package:41385089/1" override_package3d_urn="urn:adsk.eagle:package:46142980/2" override_package_urn="urn:adsk.eagle:footprint:41385037/1" value="0.1uF"/>
 <part name="GND46" library="SparkFun-PowerSymbols" library_urn="urn:adsk.eagle:library:530" deviceset="GND" device=""/>
+<part name="L4" library="LQH2MCN120K02L" deviceset="LQH2MCN120K02L" device="" value="3.3uH"/>
 </parts>
 <sheets>
@@
 <attribute name="VALUE" x="45.466" y="139.446" size="1.27" layer="96" font="vector" ratio="20" align="top-center"/>
 </instance>
-<instance part="L1" gate="G$1" x="86.36" y="129.54" smashed="yes">
-<attribute name="NAME" x="86.868" y="132.334" size="1.27" layer="95" font="vector" ratio="20"/>
-<attribute name="VALUE" x="87.122" y="124.206" size="1.27" layer="96" font="vector" ratio="20" rot="R90" align="top-left"/>
-</instance>
 <instance part="SUPPLY3" gate="G$1" x="50.8" y="132.08" smashed="yes">
 <attribute name="VALUE" x="50.8" y="134.874" size="1.27" layer="96" font="vector" ratio="20" align="bottom-center"/>
@@
 <instance part="GND41" gate="1" x="182.88" y="134.62" smashed="yes">
 <attribute name="VALUE" x="182.88" y="134.366" size="1.27" layer="96" font="vector" ratio="20" align="top-center"/>
+</instance>
+<instance part="L4" gate="G$1" x="84.074" y="128.27" smashed="yes" rot="R270">
+<attribute name="NAME" x="82.042" y="134.62" size="1.27" layer="95" font="vector" ratio="20"/>
+<attribute name="VALUE" x="81.534" y="121.158" size="1.27" layer="96" font="vector" ratio="20" align="bottom-center"/>
 </instance>
 </instances>
@@
 <wire x1="104.14" y1="134.62" x2="91.44" y2="134.62" width="0.1524" layer="91"/>
 <wire x1="91.44" y1="134.62" x2="91.44" y2="136.144" width="0.1524" layer="91"/>
-<wire x1="91.44" y1="136.144" x2="86.36" y2="136.144" width="0.1524" layer="91"/>
-<pinref part="L1" gate="G$1" pin="1"/>
-<wire x1="86.36" y1="136.144" x2="86.36" y2="134.62" width="0.1524" layer="91"/>
+<wire x1="91.44" y1="136.144" x2="84.074" y2="136.144" width="0.1524" layer="91"/>
+<pinref part="L4" gate="G$1" pin="P$1"/>
+<wire x1="84.074" y1="136.144" x2="84.074" y2="135.89" width="0.1524" layer="91"/>
 </segment>
 </net>
@@
 <wire x1="89.662" y1="132.08" x2="89.662" y2="121.158" width="0.1524" layer="91"/>
 <wire x1="89.662" y1="121.158" x2="86.36" y2="121.158" width="0.1524" layer="91"/>
-<pinref part="L1" gate="G$1" pin="2"/>
-<wire x1="86.36" y1="121.158" x2="86.36" y2="124.46" width="0.1524" layer="91"/>
 <pinref part="SUPPLY3" gate="G$1" pin="1.1V"/>
 <wire x1="50.8" y1="132.08" x2="50.8" y2="118.618" width="0.1524" layer="91"/>
@@
 <wire x1="73.152" y1="116.078" x2="73.152" y2="118.618" width="0.1524" layer="91"/>
 <junction x="73.152" y="118.618"/>
+<pinref part="L4" gate="G$1" pin="P$2"/>
+<wire x1="84.074" y1="120.65" x2="86.36" y2="120.65" width="0.1524" layer="91"/>
+<wire x1="86.36" y1="120.65" x2="86.36" y2="121.158" width="0.1524" layer="91"/>
 </segment>
 </net>
