File: Design Files/RP2040_based/citizen_science_flora_RP2040.brd (EAGLE design)
At the start: 86.6 x 79.6 mm, 118 parts, among them IC1 W25Q64JVXGIQ, J1 SM03B-SRSS-TB(LF)(SN), J2 TYPE-C-31-M-12, J4 60312202114511, J5 60312202114511, J6 TSM-102-02-S-SH, Q1 BSS138, Q2 BSS138, U1 RP2350A, U10 PCF8563T/F4,118, U11 OPS-S56AAF5, U12 OPS-S56AAF5, U13 OPS-S56AAF5, U14 OPS-S56AAF5, U15 SN74LVC1T45DBVRG4, U2 APS6404L-3SQR-ZR, U3 ESP32-C3-MINI-1-N4, U4 MIC5504-3.3YM5-T5, U5 BME690, U6 ADM3260ARSZ, U7 ENS210-LQFM, U8 SFH6325-X017TEL0631, U9 AS3935-BQFT, Y1 12MHz

Commit message: RP2040 design
Parts:
- removed C15, C16: 0.1uF, SparkFun-Capacitors:0402
- removed C18, C19: 15pF, SparkFun-Capacitors:0402
- removed L4: 3.3uH, LQH2MCN120K02L:IND_LQH2MCN120K02L
- removed R8: 1K, SparkFun-Resistors:0402
- removed U2: APS6404L-3SQR-ZR, RP2350A:APS6404L-3SQR-ZR
- removed USR_BUTTON: MOMENTARY-SWITCH-SPST-SMD-4.6X2.8MM, SparkFun-Switches:TACTILE_SWITCH_SMD_4.6X2.8MM
- removed Y1: 12MHz, SparkFun-Clocks:CRYSTAL-SMD-3.2X2.5MM
- added D3: (no value), SparkFun-LED:LED-0603
- added Q3: (no value), adafruit:NX3225
- C1, C2, C5, C6, C7, C8, C9: device SparkFun-Capacitors:0402 -> SparkFun-Capacitors:0603
- C10, C11, C14: value 4.7UF0402 -> 0.1uF; device SparkFun-Capacitors_Sai:0402 -> SparkFun-Capacitors:0603
- C12: value 4.7UF0402 -> 33pF; device SparkFun-Capacitors_Sai:0402 -> SparkFun-Capacitors:0603
- C13: value 0.1uF -> 33pF; device SparkFun-Capacitors:0402 -> SparkFun-Capacitors:0603
- C3, C4: value 0.1uF -> 1.0uF; device SparkFun-Capacitors:0402 -> SparkFun-Capacitors:0603
- R1: value 33 -> 27; device SparkFun-Resistors:0402 -> SparkFun-Resistors:0603
- R3: device SparkFun-Resistors_Sai:0402 -> SparkFun-Resistors:0603
- R4: value 27 -> 100; device SparkFun-Resistors_Sai:0402 -> SparkFun-Resistors:0603
- R7: value 10k -> 1k; device SparkFun-Resistors:0402 -> SparkFun-Resistors:0603
- U1: value RP2350A -> RP2040; device RP2350A:RP2350A -> RP2040:QFN40P700X700X90-57N
- moved R3 129.7 mm to (-53.3, -83.8), turned to 0 degrees
- moved R4 128.5 mm to (-49.5, -83.8), turned to 0 degrees
- moved C10 122.9 mm to (-49.5, -80.0), turned to 0 degrees
- moved R7 122.8 mm to (-45.7, -83.8), turned to 0 degrees
- moved C2 122.6 mm to (-53.3, -76.2), turned to 0 degrees
- moved C11 122.5 mm to (-45.7, -80.0)
- moved C12 119.6 mm to (-41.9, -80.0)
- moved C4 117.2 mm to (-45.7, -76.2)
- moved C9 116.7 mm to (-53.3, -80.0), turned to 0 degrees
- moved C13 113.9 mm to (-38.1, -80.0)
- moved R1 113.9 mm to (-30.5, -80.0), turned to 0 degrees
- moved C5 113.9 mm to (-41.9, -76.2)
- moved C6 109.5 mm to (-38.1, -76.2)
- moved C1 109.4 mm to (-33.0, -71.1), turned to 0 degrees
- moved C7 106.3 mm to (-34.3, -76.2)
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Connections:
- removed net !FLASH_CS: R7.2, U1.2, U2.1
- removed net 1.1V: C11.1, C13.1, C14.1, C15.1, L4.2, U1.23, U1.39, U1.50, U1.6
- removed net N$2: L4.1, U1.48
- removed net N$25: U1.5, USR_BUTTON.1, USR_BUTTON.2
- removed net N$7: C19.1, U1.21, Y1.1
- removed net N$8: R8.2, U1.22
- removed net USBD_N: R4.2, U1.51
- removed net USBD_P: R3.2, U1.52
- new net CLK: U1.17
- new net CS: U1.12
- new net DATA1: U1.14
- new net DATA2: U1.13
- new net INT_MOD1: U1.2
- new net INT_MOD2: U1.3
- new net N$6: R7.2, U1.21
- new net NEOPIXEL: U1.27
- new net QSPI_CS: U1.56
- new net QSPI_SCLK: U1.52
- new net QSPI_SD0: U1.53
- new net QSPI_SD1: U1.55
- new net QSPI_SD2: U1.54
- new net QSPI_SD3: U1.51
- new net SDI: U1.18
- new net SDO: U1.15
- new net SWD: U1.25
- new net USB_DM_IN: R1.1, U1.46
- new net USB_DP_IN: R3.1, U1.47
- new net VOUT: C1.1, C2.1, C3.1, U1.23, U1.45, U1.50
- new net XIN: C13.2, Q3.1, U1.20
- net !ESP32_BOOT: now also U1.30; no longer U1.31
- net !QSPI_CS: no longer U1.60
- net 3.3V: now also C10.1, C11.1, C14.1, U1.10, U1.22, U1.33, U1.42, U1.43, U1.48; no longer C1.1, C12.1, C16.1, C2.1, C3.1, R1.1, R7.1, U1.11, U1.20, U1.30, U1.38, U1.45, U1.53, U1.54, U2.8
- net BUZZER_DRIVER: no longer U1.9
- net CMD: no longer U1.19
- net DAT0: no longer U1.16
- net DAT1: no longer U1.15
- net DAT2: no longer U1.14
- net DAT3: no longer U1.17
- net ESP32_CS: now also U1.32; no longer U1.33
- net ESP32_MISO: now also U1.31; no longer U1.32
- net ESP32_RX: no longer U1.7
- net ESP32_TX: no longer U1.8
- net GND: now also C12.1, C13.1, D3.C, Q3.2, Q3.4, U1.19, U1.57; no longer C12.2, C13.2, C15.2, C16.2, C18.2, C19.2, U1.47, U1.EPAD, U2.4, U2.9, USR_BUTTON.3, USR_BUTTON.4, Y1.2, Y1.4
- net INT_RTC: now also U1.38; no longer U1.40
- net INT_SOIL: no longer U1.3
- net INT_SOILTEMP: no longer U1.4
- net IRQ_LIGHTNING: no longer U1.10
- net N$1: now also D3.A, R4.2; no longer C10.1, R1.2, U1.46
- net N$4: now also C12.2, Q3.3, R7.1; no longer C18.1, R8.1, Y1.3
- net NEOPIXEL_3.3V: no longer U1.27
- net PDIS_EN: no longer U1.12
- net QSPI_CLK: no longer U1.56, U2.6
- net SD_CLK: no longer U1.18
- net SIO0: no longer U1.57, U2.5
- net SIO1: no longer U1.59, U2.2
- net SIO2: no longer U1.58, U2.3
- net SIO3: no longer U1.55, U2.7
- net SWDIO: no longer U1.25
- net SWITCH: now also U1.16; no longer U1.13
- net USB_N: now also R1.2; no longer R4.1
- net USB_P: now also R3.2; no longer R3.1
Routing:
- net 3.3V: track 161.6 -> 98.9 mm, vias 33 -> 23
- net 1.1V: track 40.7 -> 0.00 mm, vias 4 -> 0
- net N$25: track 20.0 -> 0.00 mm
- net !FLASH_CS: track 18.1 -> 0.00 mm, vias 2 -> 0
- net QSPI_CLK: track 18.3 -> 4.65 mm, vias 2 -> 0
- net N$2: track 9.66 -> 0.00 mm
- net N$7: track 5.83 -> 0.00 mm
- net GND: track 21.6 -> 16.2 mm, vias 10 -> 9
- net USBD_P: track 5.36 -> 0.00 mm
- net USBD_N: track 5.09 -> 0.00 mm
- net N$1: track 5.06 -> 0.00 mm
- net N$8: track 3.98 -> 0.00 mm
- net N$4: track 2.77 -> 0.00 mm
- net SIO3: track 12.3 -> 10.4 mm
- net SIO1: track 22.4 -> 20.8 mm
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
Commit message: update to design files
Parts:
- added USER_BUTTON: MOMENTARY-SWITCH-SPST-SMD-4.6X2.8MM, SparkFun-Switches:TACTILE_SWITCH_SMD_4.6X2.8MM
- C1, C10, C11, C14, C2, C3, C4, C5, C6, C7, C8, C9: device SparkFun-Capacitors:0603 -> SparkFun-Capacitors_Sai:0402
- C12, C13: value 33pF -> 12pF; device SparkFun-Capacitors:0603 -> SparkFun-Capacitors_Sai:0402
- R1, R3: value 27 -> 27OHM0402; device SparkFun-Resistors:0603 -> SparkFun-Resistors_Sai:0402
- R4: value 100 -> 100OHM; device SparkFun-Resistors:0603 -> SparkFun-Resistors_Sai:0402
- R7: value 1k -> 1KOHM-0402-1/16W-1%; device SparkFun-Resistors:0603 -> SparkFun-Resistors_Sai:0402
- moved R3 129.5 mm to (13.3, 27.3), turned to 90 degrees
- moved C10 124.4 mm to (10.4, 29.0), turned to 90 degrees
- moved C9 123.4 mm to (21.0, 18.5)
- moved C3 122.5 mm to (16.1, 27.3), turned to 90 degrees
- moved C2 122.3 mm to (8.94, 29.0), turned to 90 degrees
- moved C4 121.2 mm to (17.5, 27.3), turned to 90 degrees
- moved C14 118.4 mm to (11.8, 29.0), turned to 90 degrees
- moved C6 118.1 mm to (18.9, 27.3), turned to 90 degrees
- moved R4 117.7 mm to (-1.24, 23.5), turned to 180 degrees
- moved R1 116.4 mm to (14.7, 27.3), turned to 90 degrees
- moved D3 115.4 mm to (-1.83, 25.7), turned to 90 degrees
- moved R7 112.1 mm to (13.6, 11.3), turned to 90 degrees
- moved C8 110.9 mm to (20.9, 22.1)
- moved C11 109.7 mm to (15.0, 11.3), turned to 270 degrees
- moved Q3 109.6 mm to (11.5, 11.8), turned to 270 degrees
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Connections:
- net N$6 renamed XOUT
- net USB_DM_IN renamed USBIN_N
- net USB_DP_IN renamed USBIN_P
- removed net CLK: U1.17
- removed net CS: U1.12
- removed net DATA1: U1.14
- removed net DATA2: U1.13
- removed net INT_MOD1: U1.2
- removed net INT_MOD2: U1.3
- removed net NEOPIXEL: U1.27
- removed net QSPI_CLK: IC1.6
- removed net QSPI_CS: U1.56
- removed net SDI: U1.18
- removed net SDO: U1.15
- removed net SIO0: IC1.5
- removed net SIO1: IC1.2
- removed net SIO2: IC1.3
- removed net SIO3: IC1.7
- removed net SWDIO: J1.3
- new net USR_BUTTON: U1.5, USER_BUTTON.1, USER_BUTTON.2
- new net USR_LED: R4.1, U1.2
- net !QSPI_CS: now also U1.56
- net BUZZER_DRIVER: now also U1.8
- net CMD: now also U1.18
- net DAT0: now also U1.15
- net DAT1: now also U1.14
- net DAT2: now also U1.13
- net DAT3: now also U1.16
- net ESP32_RX: now also U1.6
- net ESP32_TX: now also U1.7
- net GND: now also USER_BUTTON.3, USER_BUTTON.4
- net INT_SOIL: now also U1.3
- net INT_SOILTEMP: now also U1.4
- net IRQ_LIGHTNING: now also U1.9
- net NEOPIXEL_3.3V: now also U1.27
- net PDIS_EN: now also U1.11
- net QSPI_SCLK: now also IC1.6
- net QSPI_SD0: now also IC1.5
- net QSPI_SD1: now also IC1.2
- net QSPI_SD2: now also IC1.3
- net QSPI_SD3: now also IC1.7
- net SD_CLK: now also U1.17
- net SWD: now also J1.3
- net SWITCH: now also U1.12; no longer U1.16
Routing:
- net 3.3V: track 98.9 -> 146.1 mm, vias 23 -> 29
- net VOUT: track 0.00 -> 40.5 mm, vias 0 -> 3
- net SWDIO: track 24.2 -> 0.00 mm, vias 2 -> 0
- net SIO2: track 21.9 -> 0.00 mm, vias 3 -> 0
- net SIO1: track 20.8 -> 0.00 mm, vias 2 -> 0
- net CMD: track 54.8 -> 36.7 mm
- net SDA: track 215.9 -> 198.3 mm, vias 5 -> 4
- net !RESET: track 34.1 -> 18.4 mm, vias 2 -> 1
- net INT_SOIL: track 47.8 -> 63.2 mm
- net SWD: track 0.00 -> 15.3 mm, vias 0 -> 1
- net USR_BUTTON: track 0.00 -> 14.1 mm
- net QSPI_SD1: track 0.00 -> 13.5 mm
- net QSPI_SD2: track 0.00 -> 13.2 mm
- net SCL: track 153.7 -> 141.5 mm, vias 4 -> 3
- net !ESP32_RST: track 33.8 -> 22.5 mm, vias 2 -> 1
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
Commit message: Board design files and BoM
Parts:
- R5: value (none) -> DNF
- moved C9 0.58 mm to (21.6, 18.5)
Routing:
- net !RESET: track 18.4 -> 57.7 mm, vias 1 -> 2
- net SDA: track 198.3 -> 172.6 mm, vias 4 -> 6
- net CMD: track 36.7 -> 54.5 mm
- net !ESP32_RST: track 22.5 -> 37.4 mm, vias 1 -> 2
- net SWD: track 15.3 -> 26.0 mm, vias 1 -> 2
- net SWCLK: track 18.5 -> 29.0 mm, vias 1 -> 2
- net ESP32_MOSI: track 31.2 -> 39.1 mm, vias 1 -> 2
- net ESP32_MISO: track 29.7 -> 36.0 mm
- net ESP32_CS: track 28.6 -> 32.9 mm, vias 1 -> 2
- net !ESP32_BOOT: track 35.4 -> 39.5 mm, vias 1 -> 2
- net ESP32_HANDSHAKE: track 25.3 -> 29.4 mm, vias 1 -> 2
- net IRQ_LIGHTNING: track 56.5 -> 59.8 mm
- net 3.3V: track 146.1 -> 149.3 mm, vias 29 -> 30
- net ESP32_SCK: track 32.3 -> 35.2 mm, vias 1 -> 2
- net SCL: track 141.5 -> 140.7 mm, vias 3 -> 5
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Other:
- board text added: "Purple Daisy"
- board text added: "Purple Daisy STEAM platform"
- board text added: "RP2040"
- board text removed: "Blue Daisy"
- board text removed: "Blue Daisy STEAM platform"
- board text removed: "RP2350A"
