File: Design Files/RP2040_based/citizen_science_flora_RP2040.sch (EAGLE design)
At the start: 111 parts, among them IC1 W25Q64JVXGIQ, J1 SM03B-SRSS-TB(LF)(SN), J2 TYPE-C-31-M-12, J4 60312202114511, J5 60312202114511, J6 TSM-102-02-S-SH, Q1 BSS138, Q2 BSS138, U1 RP2040, U10 PCF8563T/F4,118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

Commit message: update to design files
Parts:
- added USER_BUTTON: MOMENTARY-SWITCH-SPST-SMD-4.6X2.8MM, SparkFun-Switches:MOMENTARY-SWITCH-SPST-SMD-4.6X2.8MM
- C1, C10, C11, C14, C2, C5, C6, C7, C8, C9: device SparkFun-Capacitors:0.1UF-0603-25V-(+80/-20%) -> SparkFun-Capacitors_Sai:0.1UF-0402-6.3V-10%-X7R
- C12, C13: value 33pF -> 12pF; device SparkFun-Capacitors:33PF-0603-50V-5% -> SparkFun-Capacitors_Sai:12PF-0402-50V-5%
- C3, C4: device SparkFun-Capacitors:1.0UF-0603-16V-10% -> SparkFun-Capacitors_Sai:1.0UF-0402-16V-10%
- R1, R3: value 27 -> 27OHM0402; device SparkFun-Resistors:27OHM-0603-1/10W-1% -> SparkFun-Resistors_Sai:27OHM0402
- R4: value 100 -> 100OHM; device SparkFun-Resistors:100OHM-0603-1/10W-1% -> SparkFun-Resistors_Sai:100OHM
- R7: value 1k -> 1KOHM-0402-1/16W-1%; device SparkFun-Resistors:1KOHM-0603-1/10W-1% -> SparkFun-Resistors_Sai:1KOHM-0402-1/16W-1%
Connections:
- net N$6 renamed XOUT
- net USB_DM_IN renamed USBIN_N
- net USB_DP_IN renamed USBIN_P
- removed net CLK: U1.GPIO14
- removed net CS: U1.GPIO9
- removed net DATA1: U1.GPIO11
- removed net DATA2: U1.GPIO10
- removed net INT_MOD1: U1.GPIO0
- removed net INT_MOD2: U1.GPIO1
- removed net NEOPIXEL: U1.GPIO16
- removed net QSPI_CLK: IC1.CLK
- removed net QSPI_CS: U1.QSPI_CSN
- removed net SDI: U1.GPIO15
- removed net SDO: U1.GPIO12
- removed net SIO0: IC1.DI(IO0)
- removed net SIO1: IC1.DO(IO1)
- removed net SIO2: IC1.!WP(IO2)
- removed net SIO3: IC1.!HOLD_OR_!RESET_(IO3)
- removed net SWDIO: J1.3
- new net USR_BUTTON: U1.GPIO3, USER_BUTTON.1
- new net USR_LED: R4.1, U1.GPIO0
- net !QSPI_CS: now also U1.QSPI_CSN
- net BUZZER_DRIVER: now also U1.GPIO6
- net CMD: now also U1.GPIO15
- net DAT0: now also U1.GPIO12
- net DAT1: now also U1.GPIO11
- net DAT2: now also U1.GPIO10
- net DAT3: now also U1.GPIO13
- net ESP32_RX: now also U1.GPIO4
- net ESP32_TX: now also U1.GPIO5
- net GND: now also USER_BUTTON.2
- net INT_SOIL: now also U1.GPIO1
- net INT_SOILTEMP: now also U1.GPIO2
- net IRQ_LIGHTNING: now also U1.GPIO7
- net NEOPIXEL_3.3V: now also U1.GPIO16
- net PDIS_EN: now also U1.GPIO8
- net QSPI_SCLK: now also IC1.CLK
- net QSPI_SD0: now also IC1.DI(IO0)
- net QSPI_SD1: now also IC1.DO(IO1)
- net QSPI_SD2: now also IC1.!WP(IO2)
- net QSPI_SD3: now also IC1.!HOLD_OR_!RESET_(IO3)
- net SD_CLK: now also U1.GPIO14
- net SWD: now also J1.3
- net SWITCH: now also U1.GPIO9; no longer U1.GPIO13

Commit message: Board design files and BoM
Parts:
- R5: value (none) -> DNF
Changed lines of the file:
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@@
 <part name="C17" library="SparkFun-Capacitors" library_urn="urn:adsk.eagle:library:510" deviceset="0.1UF" device="-0402-6.3V-10%-X7R" package3d_urn="urn:adsk.eagle:package:41385089/1" override_package3d_urn="urn:adsk.eagle:package:46143257/2" override_package_urn="urn:adsk.eagle:footprint:41385056/1" override_locally_modified="yes" value="0.1uF"/>
 <part name="GND10" library="SparkFun-PowerSymbols" library_urn="urn:adsk.eagle:library:530" deviceset="GND" device=""/>
-<part name="R5" library="SparkFun-Resistors" library_urn="urn:adsk.eagle:library:532" deviceset="RESISTOR" device="0402" package3d_urn="urn:adsk.eagle:package:39657/2" override_package3d_urn="urn:adsk.eagle:package:46141752/2" override_package_urn="urn:adsk.eagle:footprint:39625/2" value=" "/>
+<part name="R5" library="SparkFun-Resistors" library_urn="urn:adsk.eagle:library:532" deviceset="RESISTOR" device="0402" package3d_urn="urn:adsk.eagle:package:39657/2" override_package3d_urn="urn:adsk.eagle:package:46141752/2" override_package_urn="urn:adsk.eagle:footprint:39625/2" value="DNF"/>
 <part name="SUPPLY6" library="SparkFun-PowerSymbols" library_urn="urn:adsk.eagle:library:530" deviceset="3.3V" device=""/>
 <part name="R6" library="SparkFun-Resistors" library_urn="urn:adsk.eagle:library:532" deviceset="1KOHM" device="-0402-1/16W-1%" package3d_urn="urn:adsk.eagle:package:39657/2" override_package3d_urn="urn:adsk.eagle:package:46141638/3" override_package_urn="urn:adsk.eagle:footprint:39625/2" value="1K"/>
@@
 </instance>
 <instance part="R16" gate="G$1" x="31.496" y="19.812" smashed="yes">
-<attribute name="NAME" x="36.068" y="21.59" size="1.27" layer="95" font="vector" ratio="20" rot="R180" align="bottom-center"/>
+<attribute name="NAME" x="31.496" y="21.336" size="1.778" layer="95" font="vector" align="bottom-center"/>
+<attribute name="VALUE" x="31.496" y="18.288" size="1.778" layer="96" font="vector" align="top-center"/>
 </instance>
 <instance part="R17" gate="G$1" x="31.496" y="37.592" smashed="yes">
