File: Design Files/DFA_corrected/citizen_science_flora_v2_DFA_corrected.brd (EAGLE design)
At the start: 86.6 x 79.6 mm, 118 parts, among them IC1 W25Q64JVXGIQ, J1 SM03B-SRSS-TB(LF)(SN), J2 TYPE-C-31-M-12, J4 60312202114511, J5 60312202114511, J6 TSM-102-02-S-SH, Q1 BSS138, Q2 BSS138, U1 RP2350A, U10 PCF8563T/F4,118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

Commit message: via and new gerber
Added a new via and generated new gerbers
Routing:
- net GND: vias 10 -> 11
Changed lines of the file:
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@@
 <wire x1="-39.5224" y1="-6.858" x2="-39.5224" y2="-5.92" width="0.254" layer="1"/>
 <via x="-4.4196" y="-14.605" extent="1-16" drill="0.254"/>
+<via x="-28.4988" y="22.4282" extent="1-16" drill="0.254"/>
 </signal>
 <signal name="3.3V">
@@
 <wire x1="9.2635" y1="21.45" x2="9.8174" y2="21.45" width="0.1524" layer="1"/>
 <wire x1="4.2672" y1="21.9456" x2="4.2672" y2="29.4132" width="0.2032" layer="2"/>
-<via x="4.2672" y="29.4132" extent="1-16" drill="0.381"/>
+<via x="4.2672" y="29.4132" extent="1-16" drill="0.2032"/>
 <wire x1="4.3942" y1="21.8186" x2="4.2672" y2="21.9456" width="0.2032" layer="2"/>
 <wire x1="4.211" y1="28.6138" x2="4.5854" y2="28.6138" width="0.2032" layer="1"/>
